File: hardware/ws2018b.kicad_sch (KiCad schematic)
At the start: 8 parts

Commit message: All changes made, passing DRC, preparing for assembly
Parts:
- added R10: 330, Resistor_SMD:R_0402_1005Metric, symbol Device:R
- D1, D2, D3, D4, D5, D6, D7, D8: footprint LED_SMD:LED_WS2812B_PLCC4_5.0x5.0mm_P3.2mm -> ws2812b:LED_WS2812B_PLCC4_1.0x1.0mm
Connections:
- net GPIO12/NEOPIX: now also R10.1; no longer D1.4 (DIN)
- net +3V3: now reaches D8.2 (VDD)
- net +3V3: now also D1.2 (VDD), D2.2 (VDD), D3.2 (VDD), D4.2 (VDD), D5.2 (VDD), D6.2 (VDD), D7.2 (VDD)
- net GPIO11/NEO_PWR: now reaches D8.3 (VSS)
- net GPIO11/NEO_PWR: now also D1.3 (VSS), D2.3 (VSS), D3.3 (VSS), D4.3 (VSS), D5.3 (VSS), D6.3 (VSS), D7.3 (VSS)
- new net: D1.4 (DIN), R10.2
Changed lines of the file:
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@@
 (kicad_sch (version 20230121) (generator eeschema)
   (paper "A4")
-  (label "GPIO12{slash}NEOPIX" (at 59.055 55.245 180) (fields_autoplaced)
+  (junction (at 142.875 62.865) (diameter 0) (color 0 0 0 0)
+  )
+  (junction (at 127.635 47.625) (diameter 0) (color 0 0 0 0)
+  )
+  (junction (at 97.155 47.625) (diameter 0) (color 0 0 0 0)
+  )
+  (junction (at 127.635 62.865) (diameter 0) (color 0 0 0 0)
+  )
+  (junction (at 112.395 47.625) (diameter 0) (color 0 0 0 0)
+  )
+  (junction (at 158.115 47.625) (diameter 0) (color 0 0 0 0)
+  )
+  (junction (at 112.395 62.865) (diameter 0) (color 0 0 0 0)
+  )
+  (junction (at 81.915 62.865) (diameter 0) (color 0 0 0 0)
+  )
+  (junction (at 66.675 47.625) (diameter 0) (color 0 0 0 0)
+  )
+  (junction (at 97.155 62.865) (diameter 0) (color 0 0 0 0)
+  )
+  (junction (at 66.675 62.865) (diameter 0) (color 0 0 0 0)
+  )
+  (junction (at 142.875 47.625) (diameter 0) (color 0 0 0 0)
+  )
+  (junction (at 81.915 47.625) (diameter 0) (color 0 0 0 0)
+  )
+  (junction (at 158.115 62.865) (diameter 0) (color 0 0 0 0)
+  )
+  (wire (pts (xy 81.915 62.865) (xy 97.155 62.865))
+    (stroke (width 0) (type default))
+  )
+  (wire (pts (xy 142.875 47.625) (xy 158.115 47.625))
+    (stroke (width 0) (type default))
+  )
+  (wire (pts (xy 127.635 47.625) (xy 142.875 47.625))
+    (stroke (width 0) (type default))
+  )
+  (wire (pts (xy 66.675 47.625) (xy 81.915 47.625))
+    (stroke (width 0) (type default))
+  )
+  (wire (pts (xy 97.155 62.865) (xy 112.395 62.865))
+    (stroke (width 0) (type default))
+  )
+  (wire (pts (xy 81.915 47.625) (xy 97.155 47.625))
+    (stroke (width 0) (type default))
+  )
+  (wire (pts (xy 97.155 47.625) (xy 112.395 47.625))
+    (stroke (width 0) (type default))
+  )
+  (wire (pts (xy 66.675 62.865) (xy 81.915 62.865))
+    (stroke (width 0) (type default))
+  )
+  (wire (pts (xy 112.395 62.865) (xy 127.635 62.865))
+    (stroke (width 0) (type default))
+  )
+  (wire (pts (xy 158.115 62.865) (xy 173.355 62.865))
+    (stroke (width 0) (type default))
+  )
+  (wire (pts (xy 112.395 47.625) (xy 127.635 47.625))
+    (stroke (width 0) (type default))
+  )
+  (wire (pts (xy 66.675 47.625) (xy 58.42 47.625))
+    (stroke (width 0) (type default))
+  )
+  (wire (pts (xy 127.635 62.865) (xy 142.875 62.865))
+    (stroke (width 0) (type default))
+  )
+  (wire (pts (xy 142.875 62.865) (xy 158.115 62.865))
+    (stroke (width 0) (type default))
+  )
+  (wire (pts (xy 158.115 47.625) (xy 173.355 47.625))
+    (stroke (width 0) (type default))
+  )
+  (wire (pts (xy 58.42 62.865) (xy 66.675 62.865))
+    (stroke (width 0) (type default))
+  )
+  (label "GPIO12{slash}NEOPIX" (at 51.435 55.245 180) (fields_autoplaced)
     (effects (font (size 1.27 1.27)) (justify right bottom))
   )
+  (label "GPIO11{slash}NEO_PWR" (at 58.42 62.865 180) (fields_autoplaced)
+    (effects (font (size 1.27 1.27)) (justify right bottom))
+  )
   (symbol (lib_id "ws2018b:WS2812B_1x1") (at 173.355 55.245 0) (unit 1)
     (in_bom yes) (on_board yes) (dnp no) (fields_autoplaced)
@@
       (effects (font (size 1.27 1.27)))
     )
-    (property "Footprint" "LED_SMD:LED_WS2812B_PLCC4_5.0x5.0mm_P3.2mm" (at 174.625 62.865 0)
+    (property "Footprint" "ws2812b:LED_WS2812B_PLCC4_1.0x1.0mm" (at 174.625 62.865 0)
       (effects (font (size 1.27 1.27)) (justify left top) hide)
     )
@@
       (effects (font (size 1.27 1.27)))
     )
-    (property "Footprint" "LED_SMD:LED_WS2812B_PLCC4_5.0x5.0mm_P3.2mm" (at 113.665 62.865 0)
+    (property "Footprint" "ws2812b:LED_WS2812B_PLCC4_1.0x1.0mm" (at 113.665 62.865 0)
       (effects (font (size 1.27 1.27)) (justify left top) hide)
     )
@@
     )
   )
+  (symbol (lib_id "power:+3V3") (at 58.42 47.625 0) (unit 1)
+    (in_bom yes) (on_board yes) (dnp no)
+    (property "Reference" "#PWR010" (at 58.42 51.435 0)
+      (effects (font (size 1.27 1.27)) hide)
+    )
+    (property "Value" "+3V3" (at 58.801 43.2308 0)
+      (effects (font (size 1.27 1.27)))
+    )
+    (property "Footprint" "" (at 58.42 47.625 0)
+      (effects (font (size 1.27 1.27)) hide)
+    )
+    (property "Datasheet" "" (at 58.42 47.625 0)
+      (effects (font (size 1.27 1.27)) hide)
+    )
+    (pin "1")
+    (instances
+      (project "labsconbadge-23"
+        (path "/0fe9e493-c481-454c-b8b0-96af10f6ed2d"
+          (reference "#PWR010") (unit 1)
+        )
+        (path "/0fe9e493-c481-454c-b8b0-96af10f6ed2d/d12339d1-0145-4be4-b01a-e128347ab307"
+          (reference "#PWR025") (unit 1)
+        )
+      )
+      (project "RP2040_minimal"
+        (path "/a9862e0d-3ce7-4836-a3aa-a28e96dbe90c"
+          (reference "#PWR09") (unit 1)
+        )
+      )
+    )
+  )
   (symbol (lib_id "ws2018b:WS2812B_1x1") (at 81.915 55.245 0) (unit 1)
     (in_bom yes) (on_board yes) (dnp no) (fields_autoplaced)
@@
       (effects (font (size 1.27 1.27)))
     )
-    (property "Footprint" "LED_SMD:LED_WS2812B_PLCC4_5.0x5.0mm_P3.2mm" (at 83.185 62.865 0)
+    (property "Footprint" "ws2812b:LED_WS2812B_PLCC4_1.0x1.0mm" (at 83.185 62.865 0)
       (effects (font (size 1.27 1.27)) (justify left top) hide)
     )
@@
     )
   )
+  (symbol (lib_id "Device:R") (at 55.245 55.245 90) (unit 1)
+    (in_bom yes) (on_board yes) (dnp no)
+    (property "Reference" "R10" (at 55.245 60.5028 90)
+      (effects (font (size 1.27 1.27)))
+    )
+    (property "Value" "330" (at 55.245 58.1914 90)
+      (effects (font (size 1.27 1.27)))
+    )
+    (property "Footprint" "Resistor_SMD:R_0402_1005Metric" (at 55.245 57.023 90)
+      (effects (font (size 1.27 1.27)) hide)
+    )
+    (property "Datasheet" "~" (at 55.245 55.245 0)
+      (effects (font (size 1.27 1.27)) hide)
+    )
+    (property "LCSC" "C25104" (at 55.245 55.245 0)
+      (effects (font (size 1.27 1.27)) hide)
+    )
+    (property "P/N" "0402WGF3300TCE" (at 55.245 55.245 0)
+      (effects (font (size 1.27 1.27)) hide)
+    )
+    (property "Price" "$0.00" (at 55.245 55.245 0)
+      (effects (font (size 1.27 1.27)) hide)
+    )
+    (pin "1")
+    (pin "2")
+    (instances
+      (project "labsconbadge-23"
+        (path "/0fe9e493-c481-454c-b8b0-96af10f6ed2d"
+          (reference "R10") (unit 1)
+        )
+        (path "/0fe9e493-c481-454c-b8b0-96af10f6ed2d/d12339d1-0145-4be4-b01a-e128347ab307"
+          (reference "R12") (unit 1)
+        )
+      )
+      (project "RP2040_minimal"
+        (path "/a9862e0d-3ce7-4836-a3aa-a28e96dbe90c"
+          (reference "R4") (unit 1)
+        )
+      )
+    )
+  )
   (symbol (lib_id "ws2018b:WS2812B_1x1") (at 127.635 55.245 0) (unit 1)
     (in_bom yes) (on_board yes) (dnp no) (fields_autoplaced)
@@
       (effects (font (size 1.27 1.27)))
     )
-    (property "Footprint" "LED_SMD:LED_WS2812B_PLCC4_5.0x5.0mm_P3.2mm" (at 128.905 62.865 0)
+    (property "Footprint" "ws2812b:LED_WS2812B_PLCC4_1.0x1.0mm" (at 128.905 62.865 0)
       (effects (font (size 1.27 1.27)) (justify left top) hide)
     )
@@
       (effects (font (size 1.27 1.27)))
     )
-    (property "Footprint" "LED_SMD:LED_WS2812B_PLCC4_5.0x5.0mm_P3.2mm" (at 144.145 62.865 0)
+    (property "Footprint" "ws2812b:LED_WS2812B_PLCC4_1.0x1.0mm" (at 144.145 62.865 0)
       (effects (font (size 1.27 1.27)) (justify left top) hide)
     )
@@
       (effects (font (size 1.27 1.27)))
     )
-    (property "Footprint" "LED_SMD:LED_WS2812B_PLCC4_5.0x5.0mm_P3.2mm" (at 159.385 62.865 0)
+    (property "Footprint" "ws2812b:LED_WS2812B_PLCC4_1.0x1.0mm" (at 159.385 62.865 0)
       (effects (font (size 1.27 1.27)) (justify left top) hide)
     )
@@
       (effects (font (size 1.27 1.27)))
     )
-    (property "Footprint" "LED_SMD:LED_WS2812B_PLCC4_5.0x5.0mm_P3.2mm" (at 98.425 62.865 0)
+    (property "Footprint" "ws2812b:LED_WS2812B_PLCC4_1.0x1.0mm" (at 98.425 62.865 0)
       (effects (font (size 1.27 1.27)) (justify left top) hide)
     )
@@
       (effects (font (size 1.27 1.27)))
     )
-    (property "Footprint" "LED_SMD:LED_WS2812B_PLCC4_5.0x5.0mm_P3.2mm" (at 67.945 62.865 0)
-      (effects (font (size 1.27 1.27)) (justify left top) hide)
-    )
+    (property "Footprint" "ws2812b:LED_WS2812B_PLCC4_1.0x1.0mm" (at 67.945 62.865 0)
+      (effects (font (size 1.27 1.27)) (justify left top) hide)
+    )
